File: KiCad-PCB/Micro-Whirlwind-Main-PCB - As-Built Dec-2024/Analog-Scope_Interface.kicad_sch (KiCad schematic)
At the start: 22 parts, among them J1 Conn_02x08_Odd_Even, J11 Conn_01x08, J2 Conn_02x08_Odd_Even, J3 AudioJack3_Ground_SwitchTR, J4 Conn_01x03, J5 X, J6 Y, J7 Z, J8 Conn_01x03, SW25 SW_SPDT_MSM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

Commit message: I made most of the corrections to the schematic and some to the PCB. The Main PCB needs to be redone with a four-layer PCB, so I didn't re-route all the traces on the PCB The Power switch needs to be moved out of the way of the HDMI connector - that wasn't done either. See Notes/PCB-Corrections for a listing of the changes made, and the ones that are still pending   /guy
Parts:
- RV1, RV2, RV3: footprint mWW-Project-Library:Potentiometer_Bourns_PTV09A-2_Single_Horizontal -> Potentiometer_THT:Potentiometer_Bourns_PTV09A-2_Single_Horizontal; symbol mWW_Library:R_Potentiometer -> Device:R_Potentiometer
- SW25: symbol mWW_Library:SW_SPDT_MSM -> Switch:SW_SPDT_MSM
Connections:
- net +5V-Unswitched is gone; now on net +5V: J2.9 (Pin_9)
- net GND: no longer RV1.4 (GND), RV2.4 (GND), RV3.4 (GND), SW25.4 (GND)
- net GPIO_Audio: now also J11.4 (Pin_4), RV3.3; no longer C9.1
- net at J3.R, J3.T, R12.2: now also C9.2; no longer R7.1
- new net: C9.1, R7.1
Other:
- note removed: "Connector from ADC Board"
- note removed: "External TAP Cpnnector"
- note removed: "Grounded switch frame"
- moved on the sheet: C9
