File: KiCad-PCB/Micro-Whirlwind-Main-PCB - As-Built Dec-2024/Micro-Whirlwind-Main-PCB.kicad_pcb (KiCad board)
At the start: 2 copper layers, 210 x 279 mm, 145 parts, among them J1 Conn_02x08_Odd_Even, J11 Conn_01x08, J2 Conn_02x08_Odd_Even, J3 AudioJack3_Ground_SwitchTR, J4 Conn_01x03, J5 X, J6 Y, J7 Z, J8 Conn_01x03, J9 RaspiGPIO40, Q1 IRF5305, Q2 BSS138, Q5 BSS138, SW1 mSW_Push_LEDx8, SW10 SW_Push_LED, SW11 SW_Push_LED, SW12 SW_Push_LED, SW13 SW_Push_LED, SW14 SW_Push_LED, SW15 SW_Push_LED, SW18 mSW_Push_LEDx8, SW19 mSW_Push_LEDx8, SW2 mSW_Push_LEDx8, SW20 mSW_Push_LEDx8, SW21 mSW_Push_LEDx8, SW22 mSW_Push_LEDx8, SW23 SW_Push_LED, SW24 SW_Push_LED, SW25 SW_SPDT_MSM, SW28 SW_Push_LED, SW29 SW_Push_LED, SW3 mSW_Push_LEDx8, SW30 SW_Push_LED, SW31 SW_Push_LED, SW32 SW_Push_LED, SW33 SW_Push_LED, SW34 SW_Push_LED, SW35 SW_Push_LED, SW36 SW_Push_LED, SW37 SW_Push_LED, SW38 SW_Push_LED, SW39 SW_Push_LED, SW4 mSW_Push_LEDx8, SW40 SW_Push_LED, SW5 mSW_Push_LEDx8, SW6 SW_Push_LED, SW7 SW_Push_LED, SW8 SW_Push_LED, SW9 SW_Push_LED, U1 IS31FL3731-SA, U10 4001, U2 IS31FL3731-SA, U3 TCA8418RTWR, U4 TCA8418RTWR, U5 IS31FL3731-SA, U6 LTC4316IDD_PBF, U8 RasPi Outline, U9 D_to_A_Outline

Commit message: I made most of the corrections to the schematic and some to the PCB. The Main PCB needs to be redone with a four-layer PCB, so I didn't re-route all the traces on the PCB The Power switch needs to be moved out of the way of the HDMI connector - that wasn't done either. See Notes/PCB-Corrections for a listing of the changes made, and the ones that are still pending   /guy
Parts:
- removed R13, R14: 3.3K, mWW-Project-Library:SM-1206B
- L1: footprint mWW-Project-Library:Logo-Large -> mWW-Project-Library:Logo
- R17: value 22K -> 1K
- R18: value 1.5K -> 470
- RV1, RV2, RV3: footprint mWW-Project-Library:Potentiometer_Bourns_PTV09A-2_Single_Horizontal -> Potentiometer_THT:Potentiometer_Bourns_PTV09A-2_Single_Horizontal
- turned R11 to 90 degrees
Connections:
- net /Analog-Scope_Interface/GPIO_Audio_Sync renamed GPIO_Audio_Sync
- C9 pad 1: /Analog-Scope_Interface/GPIO_Audio -> Net-(C9-Pad1)
- C9 pad 2: Net-(J11-Pin_4) -> Net-(C9-Pad2)
- F1 pad 1: /Analog-Scope_Interface/+5V-Unswitched -> Net-(Q1-S)
- J11 pad 4: Net-(J11-Pin_4) -> GPIO_Audio
- J2 pad 9: /Analog-Scope_Interface/+5V-Unswitched -> +5V
- J3 pad R: Net-(J3-PadR) -> Net-(C9-Pad2)
- J3 pad T: Net-(J3-PadR) -> Net-(C9-Pad2)
- J9 pad 32: /Analog-Scope_Interface/GPIO_Audio -> /SpareGPIO
- Q1 pad 3: /Analog-Scope_Interface/+5V-Unswitched -> Net-(Q1-S)
- Q2 pad 3: /Analog-Scope_Interface/+5V-Unswitched -> Net-(Q1-S)
- R12 pad 2: Net-(J3-PadR) -> Net-(C9-Pad2)
- R15 pad 1: /Analog-Scope_Interface/+5V-Unswitched -> Net-(Q1-S)
- R7 pad 1: Net-(J3-PadR) -> Net-(C9-Pad1)
- RV3 pad 3: Net-(J11-Pin_4) -> GPIO_Audio
- U3 pad 22: /SDA_3V3 -> /SCL_3V3
- U3 pad 23: /SCL_3V3 -> /SDA_3V3
- U4 pad 22: /Execution-Control/SDA_3V3 -> /Execution-Control/SCL_3V3
- U4 pad 23: /Execution-Control/SCL_3V3 -> /Execution-Control/SDA_3V3
Routing:
- net Net-(J11-Pin_4): track 324.8 -> 0.00 mm, vias 2 -> 0
- net GPIO_Audio: track 0.00 -> 324.8 mm, vias 0 -> 2
- net /Analog-Scope_Interface/+5V-Unswitched: track 257.3 -> 0.00 mm
- net Net-(Q1-S): track 0.00 -> 257.0 mm
- net (no net): track 52.9 -> 0.00 mm
- net Net-(C9-Pad2): track 0.00 -> 44.9 mm
- net GND: track 1013.5 -> 1004.3 mm
- net +3.3V: track 344.5 -> 336.1 mm
- net Net-(C9-Pad1): track 0.00 -> 8.00 mm
- net /Execution-Control/SCL_3V3: track 168.1 -> 161.4 mm, vias 8 -> 6
- net /Execution-Control/SDA_3V3: track 170.6 -> 163.9 mm, vias 7 -> 6
- net Net-(J7-In): track 11.4 -> 17.7 mm, vias 0 -> 1
- net /MIR-Switches/MIR-B5: track 542.0 -> 538.6 mm
- net Net-(J5-In): track 20.6 -> 17.9 mm, vias 1 -> 0
- net Net-(J6-In): track 17.3 -> 15.0 mm, vias 1 -> 0
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