File: KiCad-PCB/Micro-Whirlwind-Main-PCB - As-Built Dec-2024/Micro-Whirlwind-Main-PCB.kicad_sch (KiCad schematic)
At the start: 36 parts, among them J9 RaspiGPIO40, Q1 IRF5305, Q2 BSS138, Q5 BSS138, U6 LTC4316IDD_PBF, U8 RasPi Outline, U9 D_to_A_Outline

Commit message: I made most of the corrections to the schematic and some to the PCB. The Main PCB needs to be redone with a four-layer PCB, so I didn't re-route all the traces on the PCB The Power switch needs to be moved out of the way of the HDMI connector - that wasn't done either. See Notes/PCB-Corrections for a listing of the changes made, and the ones that are still pending   /guy
Parts:
- removed R13, R14: 3.3K, mWW-Project-Library:SM-1206B, symbol Device:R
- R17: value 22K -> 1K
- R18: value 1.5K -> 470
Connections:
- net Analog-Scope_Interface/+5V-Unswitched: no longer names the net of F1.1, Q1.3 (S), Q2.3 (D), R15.1
- net Analog-Scope_Interface/GPIO_Audio renamed SpareGPIO
- no-connect marks 22 -> 23
Other:
- sheet Analog-Scope_Interface ports: added none; removed +5V-Unswitched, GPIO_Audio, GPIO_Audio_Sync
- note removed: "This connection picks up a second +5 Unswitched signal from the DAC board"
- moved on the sheet: C10, C11, C4, C5, C6, C7, C8, D14, F1, H1, H2, H3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
