File: KiCad-PCB/Micro-Whirlwind-Main-PCB/Execution-Control.kicad_sch (KiCad schematic)
At the start: 15 parts, among them SW28 SW_Push_LED, SW29 SW_Push_LED, SW30 SW_Push_LED, SW31 SW_Push_LED, SW32 SW_Push_LED, SW33 SW_Push_LED, SW34 SW_Push_LED, SW35 SW_Push_LED, SW36 SW_Push_LED, SW37 SW_Push_LED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

Commit message: added one new LED to indicate that the Light Gun is active.  See page 'Execution Control'
Parts:
- added D19: LED, LED_THT:LED_D3.0mm, symbol Device:LED
Connections:
- net MIR-B6: now also D19.2 (A)
- net MIR-B8: now also D19.1 (K)
Other:
- note added: "D-Scope U2_led[7] bit 12"
- note added: "F-Scope U2_led[7] bit 11"
- note added: "Light-Gun Active U2_led[7] bit 13 added Jun 14, 2026"
- note removed: "D-Scope"
- note removed: "F-Scope"
Changed lines of the file:
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@@
 	(generator_version "9.0")
 	(paper "B")
-	(text "F-Scope"
+	(text "F-Scope\nU2_led[7] bit 11"
 		(exclude_from_sim no)
-		(at 239.776 93.218 0)
+		(at 243.586 92.964 0)
 		(effects
 			(font
@@
 		)
 	)
+	(text "Light-Gun Active\nU2_led[7] bit 13\nadded Jun 14, 2026"
+		(exclude_from_sim no)
+		(at 246.126 129.794 0)
+		(effects
+			(font
+				(size 1.27 1.27)
+			)
+		)
+	)
 	(text "TCA8418 has a fixed I2C address \nof 0x34.  No way to change!"
 		(exclude_from_sim yes)
@@
 		)
 	)
-	(text "D-Scope"
+	(text "D-Scope\nU2_led[7] bit 12"
 		(exclude_from_sim no)
-		(at 239.776 112.268 0)
+		(at 243.586 111.76 0)
 		(effects
 			(font
@@
 	)
 	(junction
+		(at 215.9 129.54)
+		(diameter 0)
+		(color 0 0 0 0)
+	)
+	(junction
 		(at 213.36 90.17)
 		(diameter 0)
@@
 		(color 0 0 0 0)
 	)
+	(junction
+		(at 198.12 134.62)
+		(diameter 0)
+		(color 0 0 0 0)
+	)
 	(no_connect
 		(at 279.4 185.42)
@@
 	(wire
 		(pts
+			(xy 232.41 129.54) (xy 232.41 134.62)
+		)
+		(stroke
+			(width 0)
+			(type default)
+		)
+	)
+	(wire
+		(pts
 			(xy 163.83 96.52) (xy 163.83 48.26)
 		)
@@
 	(wire
 		(pts
+			(xy 215.9 129.54) (xy 215.9 151.13)
+		)
+		(stroke
+			(width 0)
+			(type default)
+		)
+	)
+	(wire
+		(pts
 			(xy 279.4 190.5) (xy 213.36 190.5)
 		)
@@
 	(wire
 		(pts
+			(xy 229.87 129.54) (xy 232.41 129.54)
+		)
+		(stroke
+			(width 0)
+			(type default)
+		)
+	)
+	(wire
+		(pts
 			(xy 237.49 99.06) (xy 237.49 109.22)
 		)
@@
 	(wire
 		(pts
+			(xy 215.9 129.54) (xy 222.25 129.54)
+		)
+		(stroke
+			(width 0)
+			(type default)
+		)
+	)
+	(wire
+		(pts
 			(xy 205.74 156.21) (xy 238.76 156.21)
 		)
@@
 	(wire
 		(pts
-			(xy 215.9 111.76) (xy 215.9 151.13)
+			(xy 215.9 111.76) (xy 215.9 129.54)
 		)
 		(stroke
@@
 	(wire
 		(pts
+			(xy 232.41 134.62) (xy 198.12 134.62)
+		)
+		(stroke
+			(width 0)
+			(type default)
+		)
+	)
+	(wire
+		(pts
 			(xy 360.68 73.66) (xy 360.68 128.27)
 		)
@@
 					(unit 1)
 				)
+			)
+		)
+	)
+	(symbol
+		(lib_id "Device:LED")
+		(at 226.06 129.54 0)
+		(unit 1)
+		(exclude_from_sim no)
+		(in_bom yes)
+		(on_board yes)
+		(dnp no)
+		(property "Reference" "D19"
+			(at 225.552 127 0)
+			(effects
+				(font
+					(size 1.27 1.27)
+				)
+			)
+		)
+		(property "Value" "LED"
+			(at 229.616 128.27 0)
+			(effects
+				(font
+					(size 1.27 1.27)
+				)
+			)
+		)
+		(property "Footprint" "LED_THT:LED_D3.0mm"
+			(at 226.06 129.54 0)
+			(effects
+				(font
+					(size 1.27 1.27)
+				)
+				(hide yes)
+			)
+		)
+		(property "Datasheet" "~"
+			(at 226.06 129.54 0)
+			(effects
+				(font
+					(size 1.27 1.27)
+				)
+				(hide yes)
+			)
+		)
+		(property "Description" "Light emitting diode"
+			(at 226.06 129.54 0)
+			(effects
+				(font
+					(size 1.27 1.27)
+				)
+				(hide yes)
+			)
+		)
+		(pin "2"
+		)
+		(pin "1"
+		)
+		(instances
+			(project "Micro-Whirlwind-Main-PCB"
+				(path "/83dfe2c9-ab1a-4178-9feb-71b29481afb4/aba83ce9-7044-4816-b03c-463b3738e5e7"
+					(reference "D19")
+					(unit 1)
+				)
